Commit message: Added wall and simulation with gazebo and hil. Needs to test with HIL

File: hku_m100_description/urdf/hku_m100_base_with_gimbal.urdf.xacro (robot description, xacro)
@@ -9,5 +9,5 @@
     <link name="base_link">
       <inertial>
-        <mass value="1.477" />
+        <mass value="2.477" />
         <origin xyz="0 0 0" />
         <inertia ixx="0.01152" ixy="0.0" ixz="0.0" iyy="0.01152" iyz="0.0" izz="0.0218" />
@@ -63,4 +63,9 @@
   </xacro:gimbal_camera>
  -->
+<!-- ###################################################################################################### -->
+<!-- ###################################################################################################### -->
+<!-- HOKUYO -->
+<!-- ###################################################################################################### -->
+<!-- ###################################################################################################### -->
     <joint name="laser_joint" type="fixed">
       <origin xyz="0.1 0 0.125" rpy="0 0 0" />
@@ -90,13 +95,13 @@
         <scan>
           <horizontal>
-            <samples>1080</samples>
-            <resolution>0.25</resolution>
-            <min_angle>-2.3561945</min_angle>
-            <max_angle>2.3561945</max_angle>
+            <samples>1081</samples>
+            <!-- <resolution>0.25</resolution> -->
+            <min_angle>-2.35619449615</min_angle>
+            <max_angle>2.35619449615</max_angle>
           </horizontal>
         </scan>
         <range>
           <min>0.10</min>
-          <max>30.0</max>
+          <max>10.0</max>
           <resolution>0.01</resolution>
         </range>
@@ -117,4 +122,9 @@
     </sensor>
   </gazebo>
+<!-- ###################################################################################################### -->
+<!-- ###################################################################################################### -->
+<!-- CAMERA -->
+<!-- ###################################################################################################### -->
+<!-- ###################################################################################################### -->
    <joint name="camera_joint" type="floating">
       <origin xyz="0.1 0 -0.04" rpy="0 0 0"/>
@@ -154,9 +164,10 @@
           <!-- <pose>0.027 0 -0.027 0 1.57 0</pose> -->
           <pose>0.027 0 -0.027 0 0 0</pose>
-          <horizontal_fov>${94 * M_PI/180.0}</horizontal_fov>
+          <horizontal_fov>${64.5 * M_PI/180.0}</horizontal_fov>
+          <!-- <vertical_fov>${46.6 * M_PI/180.0}</vertical_fov> -->
           <image>
             <format>R8G8B8</format>
-            <width>640</width>
-            <height>480</height>
+            <width>1280</width>
+            <height>720</height>
           </image>
           <clip>
@@ -169,6 +180,6 @@
           <alwaysOn>true</alwaysOn>
           <updateRate>30</updateRate>
-          <imageTopicName>/dji_sdk/image_raw</imageTopicName>
-          <cameraInfoTopicName>/dji_sdk/camera_info</cameraInfoTopicName>
+          <imageTopicName>/camera/image_raw</imageTopicName>
+          <cameraInfoTopicName>/camera/camera_info</cameraInfoTopicName>
           <!-- <imageTopicName>camera/image</imageTopicName> -->
           <!-- <cameraInfoTopicName>camera/camera_info</cameraInfoTopicName> -->

Commit message: First commit after days of random laser testing

File: hku_m100_description/urdf/hku_m100_base_with_gimbal.urdf.xacro (robot description, xacro)
@@ -7,5 +7,5 @@
  <!-- Main quadrotor link -->
   <xacro:macro name="hku_m100_base_macro">
-    <link name="base_link">
+    <link name="drone"> <!-- base_link -->
       <inertial>
         <mass value="2.477" />
@@ -13,5 +13,5 @@
         <inertia ixx="0.01152" ixy="0.0" ixz="0.0" iyy="0.01152" iyz="0.0" izz="0.0218" />
       </inertial>
-      <visual>
+      <!-- <visual>
         <origin xyz="0 0 0" rpy="0 0 0" />
         <geometry>
@@ -24,5 +24,5 @@
           <mesh filename="package://hku_m100_description/meshes/hku_m100/hku_m100.stl"/>
         </geometry>
-      </collision>
+      </collision> -->
     </link>
     <!-- Sonar height sensor -->
@@ -69,11 +69,13 @@
 <!-- ###################################################################################################### -->
     <joint name="laser_joint" type="fixed">
-      <origin xyz="0.1 0 0.125" rpy="0 0 0" />
-      <parent link="base_link" />
+      <origin xyz="0 0 0" rpy="0 0 0" />
+      <!-- <origin xyz="0.1 0 0.125" rpy="0 0 0" />  -->
+      <parent link="drone" />
       <child link="hokuyo_link" />
     </joint>
     <link name="hokuyo_link">
       <visual>
-        <origin xyz="0 0 -0.03" rpy="0 0 0"/>
+        <!-- <origin xyz="0 0 -0.03" rpy="0 0 0"/> -->
+        <origin xyz="0 0 0" rpy="0 0 0"/>
         <geometry>
           <box size="0.065 0.065 0.07"/>
@@ -113,5 +115,5 @@
                reading. -->
           <mean>0.0</mean>
-          <stddev>0.01</stddev>
+          <stddev>0.001</stddev>
         </noise>
       </ray>
@@ -127,7 +129,7 @@
 <!-- ###################################################################################################### -->
 <!-- ###################################################################################################### -->
-   <joint name="camera_joint" type="floating">
+    <joint name="camera_joint" type="floating">
       <origin xyz="0.1 0 -0.04" rpy="0 0 0"/>
-      <parent link="base_link"/>
+      <parent link="drone"/>
       <child link="camera_link"/>
     </joint>
@@ -151,10 +153,10 @@
       </collision>
     </link>
-    <joint name="camera_optical_joint" type="floating">
+    <!-- <joint name="camera_optical_joint" type="floating">
       <origin xyz="0 0 0" rpy="${-M_PI/2} 0.0 ${-M_PI/2}" />
       <parent link="camera_link" />
       <child link="camera_optical_frame"/>
     </joint>
-    <link name="camera_optical_frame"/>
+    <link name="camera_optical_frame"/> -->
     <gazebo reference="camera_link">
       <sensor type="camera" name="camera_camera_sensor">
