Commit message: Fixed laser and camera position calculations using correct tf transforming and sensor position offset

File: hku_m100_description/urdf/hokuyo_w_camera.urdf.xacro (robot description, xacro)
@@ -13,54 +13,5 @@
         <inertia ixx="0.01152" ixy="0.0" ixz="0.0" iyy="0.01152" iyz="0.0" izz="0.0218" />
       </inertial>
-      <visual>
-        <origin xyz="0 0 0" rpy="0 0 0" />
-        <geometry>
-          <mesh filename="package://hku_m100_description/meshes/hku_m100/hku_m100.dae"/>
-        </geometry>
-      </visual>
-      <collision>
-        <origin xyz="0 0 0" rpy="0 0 0" />
-        <geometry>
-          <mesh filename="package://hku_m100_description/meshes/hku_m100/hku_m100.stl"/>
-        </geometry>
-      </collision>
     </link>
-    <!-- Sonar height sensor -->
-     <!--<xacro:sonar_sensor name="sonar" parent="base_link" ros_topic="sonar_height" update_rate="10" min_range="0.03" max_range="3.0" field_of_view="${40*pi/180}" ray_count="3">
-      <origin xyz="-0.16 0.0 -0.012" rpy="0 ${90*pi/180} 0"/>
-    </xacro:sonar_sensor>-->
-    <!-- Camera -->
-    <!-- <link name="camera_link">
-    <collision>
-      <origin xyz="0 0 0" rpy="0 0 0"/>
-      <geometry>
-        <mesh filename="package://hku_m100_description/meshes/hku_m100/gimbal.dae"/>
-      </geometry>
-    </collision>
-    <visual>
-      <origin xyz="0 0 0" rpy="0 0 0"/>
-      <geometry>
-        <mesh filename="package://hku_m100_description/meshes/hku_m100/gimbal.stl"/>
-      </geometry>
-    </visual>
-    <inertial>
-      <mass value="1e-5" />
-      <origin xyz="0 0 0" rpy="0 0 0"/>
-      <inertia ixx="1e-6" ixy="0" ixz="0" iyy="1e-6" iyz="0" izz="1e-6" />
-    </inertial>
-  </link>
-  <joint name="camera_joint" type="fixed">
-    <axis xyz="0 1 0" />
-    <origin xyz="$0 0 0" rpy="0 0 0"/>
-    <parent link="base_link"/>
-    <child link="camera_link"/>
-  </joint>
- -->
-  <!-- <xacro:include filename="$(find hku_m100_description)/urdf/hku_m100.gazebo" /> -->
-<!--   <xacro:include filename="$(find hku_m100_description)/urdf/gimbal_camera.urdf.xacro"/>
-  <xacro:gimbal_camera name="camera" parent="base_link" ros_topic="camera/image" cam_info_topic="camera/camera_info" update_rate="10" res_x="320" res_y="240" image_format="R8G8B8" hfov="90">
-    <origin xyz="0.05 0.0 -0.06" rpy="0 0 0"/>
-  </xacro:gimbal_camera>
- -->
 <!-- ###################################################################################################### -->
 <!-- ###################################################################################################### -->
@@ -76,6 +27,6 @@
     <link name="hokuyo_link">
       <visual>
-        <origin xyz="0 0 -0.03" rpy="0 0 0"/>
-        <!-- <origin xyz="0 0 0" rpy="0 0 0"/> -->
+        <!-- <origin xyz="0 0 -0.03" rpy="0 0 0"/> -->
+        <origin xyz="0 0 0" rpy="0 0 0"/>
         <geometry>
           <box size="0.065 0.065 0.07"/>
@@ -166,5 +117,5 @@
           <!-- <pose>0.027 0 -0.027 0 1.57 0</pose> -->
           <pose>0.027 0 -0.027 0 0 0</pose>
-          <horizontal_fov>${64.5 * M_PI/180.0}</horizontal_fov>
+          <horizontal_fov>${61 * M_PI/180.0}</horizontal_fov>
           <!-- <vertical_fov>${46.6 * M_PI/180.0}</vertical_fov> -->
           <image>
@@ -182,5 +133,5 @@
           <alwaysOn>true</alwaysOn>
           <updateRate>30</updateRate>
-          <focal_length>1070</focal_length>
+          <!-- <focal_length>1070</focal_length> -->
           <imageTopicName>/usb_cam/image_raw</imageTopicName>
           <cameraInfoTopicName>/usb_cam/camera_info</cameraInfoTopicName>
